Commit message: metal.launch

File: hyperlync_simulator_2/hyperlync_robot/robot_description/urdf/andbot.xacro (robot description, xacro)
@@ -21,5 +21,5 @@
       <origin xyz="0 0 -0.019" rpy="1.57 0 -1.57"/>
       <geometry>
-        <mesh filename="package://andbot_gazebo/robot_description/mesh/lidar_XV-11.STL"/>
+        <mesh filename="package://hyperlync_robot/robot_description/mesh/lidar_XV-11.STL"/>
       </geometry>
     </collision>
@@ -27,5 +27,5 @@
       <origin xyz="0 0 -0.019" rpy="1.57 0 -1.57"/>
       <geometry>
-        <mesh filename="package://andbot_gazebo/robot_description/mesh/lidar_XV-11.STL"/>
+        <mesh filename="package://hyperlync_robot/robot_description/mesh/lidar_XV-11.STL"/>
       </geometry>
        <material name="Green">
@@ -46,11 +46,11 @@
     <child link="xv11"/>
 <!--    plastic model     -->
-<!--	<origin xyz="-0.022 0 ${radius_wheel+0.135}" rpy="0 0 0"/>	-->
+<origin xyz="-0.022 0 ${radius_wheel+0.135}" rpy="0 0 0"/>
 <!--	metal model	-->
-<origin xyz="0.07 0 ${radius_wheel+0.135}" rpy="0 0 0"/>
+<!--	<origin xyz="0.07 0 ${radius_wheel+0.135}" rpy="0 0 0"/>-->
   </joint>
 <joint name="IMU_joint" type="fixed">
     <axis xyz="1 0 0"/>
-        <origin xyz="-0.2 0.15 0.055"/>
+        <origin xyz="0.0 0.0 0.055"/>
 	    <parent link="base_link"/>
 	    <child link="IMU_link"/>
@@ -81,5 +81,5 @@
       <origin xyz="0 0 ${radius_wheel-height_wheels_from_base}" rpy="0 0 0"/>
       <geometry>
-        <mesh filename="package://andbot_gazebo/robot_description/mesh/base_part.STL"/>
+        <mesh filename="package://hyperlync_robot/robot_description/mesh/base_part.STL"/>
       </geometry>
     </collision>
@@ -87,5 +87,5 @@
       <origin xyz="0 0 ${radius_wheel-height_wheels_from_base}" rpy="0 0 0"/>
       <geometry>
-        <mesh filename="package://andbot_gazebo/robot_description/mesh/base_part.STL"/>
+        <mesh filename="package://hyperlync_robot/robot_description/mesh/base_part.STL"/>
       </geometry>
        <material name="Orange">
@@ -147,11 +147,11 @@
       <origin xyz="0 0 0" rpy="0 0 0"/>
       <geometry>
-        <mesh filename="package://andbot_gazebo/robot_description/mesh/fake_body.STL"/>
-      </geometry>
-    </collision>
-    <visual>
-      <origin xyz="0 0 0" rpy="0 0 0"/>
-      <geometry>
-        <mesh filename="package://andbot_gazebo/robot_description/mesh/fake_body.STL"/>
+        <mesh filename="package://hyperlync_robot/robot_description/mesh/fake_body.STL"/>
+      </geometry>
+    </collision>
+    <visual>
+      <origin xyz="0 0 0" rpy="0 0 0"/>
+      <geometry>
+        <mesh filename="package://hyperlync_robot/robot_description/mesh/fake_body.STL"/>
       </geometry>
        <material name="Blue">
@@ -178,11 +178,11 @@
       <origin xyz="0 0 0" rpy="0 0 0"/>
       <geometry>
-        <mesh filename="package://andbot_gazebo/robot_description/mesh/head.STL"/>
-      </geometry>
-    </collision>
-    <visual>
-      <origin xyz="0 0 0" rpy="0 0 0"/>
-      <geometry>
-        <mesh filename="package://andbot_gazebo/robot_description/mesh/head.STL"/>
+        <mesh filename="package://hyperlync_robot/robot_description/mesh/head.STL"/>
+      </geometry>
+    </collision>
+    <visual>
+      <origin xyz="0 0 0" rpy="0 0 0"/>
+      <geometry>
+        <mesh filename="package://hyperlync_robot/robot_description/mesh/head.STL"/>
       </geometry>
        <material name="Blue">
@@ -224,5 +224,5 @@
       <origin xyz="0 0 0" rpy="-1.5707 1.5707 0"/>
       <geometry>
-        <mesh filename="package://andbot_gazebo/robot_description/mesh/arm_link1.STL"/>
+        <mesh filename="package://hyperlync_robot/robot_description/mesh/arm_link1.STL"/>
       </geometry>
     </collision>
@@ -230,5 +230,5 @@
       <origin xyz="0 0 0" rpy="-1.5707 1.5707 0"/>
       <geometry>
-        <mesh filename="package://andbot_gazebo/robot_description/mesh/arm_link1.STL"/>
+        <mesh filename="package://hyperlync_robot/robot_description/mesh/arm_link1.STL"/>
       </geometry>
        <material name="Blue">
@@ -256,5 +256,5 @@
       <origin xyz="0 0 0" rpy="-1.5707 1.5707 0"/>
       <geometry>
-        <mesh filename="package://andbot_gazebo/robot_description/mesh/arm_link2.STL"/>
+        <mesh filename="package://hyperlync_robot/robot_description/mesh/arm_link2.STL"/>
       </geometry>
     </collision>
@@ -262,5 +262,5 @@
       <origin xyz="0 0 0" rpy="-1.5707 1.5707 0"/>
       <geometry>
-        <mesh filename="package://andbot_gazebo/robot_description/mesh/arm_link2.STL"/>
+        <mesh filename="package://hyperlync_robot/robot_description/mesh/arm_link2.STL"/>
       </geometry>
        <material name="Blue">
@@ -288,5 +288,5 @@
       <origin xyz="0 0 0" rpy="1.57 1.5707 0"/>
       <geometry>
-        <mesh filename="package://andbot_gazebo/robot_description/mesh/arm_link1.STL"/>
+        <mesh filename="package://hyperlync_robot/robot_description/mesh/arm_link1.STL"/>
       </geometry>
     </collision>
@@ -294,5 +294,5 @@
       <origin xyz="0 0 0" rpy="1.57 1.5707 0"/>
       <geometry>
-        <mesh filename="package://andbot_gazebo/robot_description/mesh/arm_link1.STL"/>
+        <mesh filename="package://hyperlync_robot/robot_description/mesh/arm_link1.STL"/>
       </geometry>
        <material name="Blue">
@@ -320,5 +320,5 @@
       <origin xyz="0 0 0" rpy="-1.5707 1.5707 3.14"/>
       <geometry>
-        <mesh filename="package://andbot_gazebo/robot_description/mesh/arm_link2.STL"/>
+        <mesh filename="package://hyperlync_robot/robot_description/mesh/arm_link2.STL"/>
       </geometry>
     </collision>
@@ -326,5 +326,5 @@
       <origin xyz="0 0 0" rpy="-1.5707 1.5707 0"/>
       <geometry>
-        <mesh filename="package://andbot_gazebo/robot_description/mesh/arm_link2.STL"/>
+        <mesh filename="package://hyperlync_robot/robot_description/mesh/arm_link2.STL"/>
       </geometry>
        <material name="Blue">
@@ -384,5 +384,5 @@
       <origin xyz="0 0 0" rpy="0 1.570795 1.570795"/>
       <geometry>
-        <mesh filename="package://andbot_gazebo/robot_description/mesh/wheel-D152_SMALL.STL"/>
+        <mesh filename="package://hyperlync_robot/robot_description/mesh/wheel-D152_SMALL.STL"/>
       </geometry>
     </collision>
@@ -390,5 +390,5 @@
       <origin xyz="0 0 0" rpy="0 1.570795 1.570795"/>
       <geometry>
-        <mesh filename="package://andbot_gazebo/robot_description/mesh/wheel-D152_SMALL.STL"/>
+        <mesh filename="package://hyperlync_robot/robot_description/mesh/wheel-D152_SMALL.STL"/>
       </geometry>
        <material name="Black">
@@ -435,5 +435,5 @@
       <origin xyz="0 0 0" rpy="0 1.570795 1.570795"/>
       <geometry>
-        <mesh filename="package://andbot_gazebo/robot_description/mesh/wheel-D152_SMALL.STL"/>
+        <mesh filename="package://hyperlync_robot/robot_description/mesh/wheel-D152_SMALL.STL"/>
       </geometry>
     </collision>
@@ -441,5 +441,5 @@
       <origin xyz="0 0 0" rpy="0 1.570795 1.570795"/>
       <geometry>
-        <mesh filename="package://andbot_gazebo/robot_description/mesh/wheel-D152_SMALL.STL"/>
+        <mesh filename="package://hyperlync_robot/robot_description/mesh/wheel-D152_SMALL.STL"/>
       </geometry>
        <material name="Black">
@@ -486,5 +486,5 @@
     <parent link="base_link"/>
     <child link="sonar_1"/>
-    <origin xyz="-0.10374 0.23695 ${0.03475+0.029}"  rpy="0 0 1.5707"/>
+    <origin xyz="0.15 0 ${0.03475+0.029}" rpy="0 0 0"/>
   </joint>
 <!--Sonar Link1-->
@@ -493,11 +493,11 @@
       <origin xyz="0 0 0" rpy="0 0 0"/>
       <geometry>
-        <mesh filename="package://andbot_gazebo/robot_description/mesh/sonar_HC_SR04.STL"/>
-      </geometry>
-    </collision>
-    <visual>
-      <origin xyz="0 0 0" rpy="0 0 0"/>
-      <geometry>
-        <mesh filename="package://andbot_gazebo/robot_description/mesh/sonar_HC_SR04.STL"/>
+        <mesh filename="package://hyperlync_robot/robot_description/mesh/sonar_HC_SR04.STL"/>
+      </geometry>
+    </collision>
+    <visual>
+      <origin xyz="0 0 0" rpy="0 0 0"/>
+      <geometry>
+        <mesh filename="package://hyperlync_robot/robot_description/mesh/sonar_HC_SR04.STL"/>
       </geometry>
        <material name="Yellow">
@@ -523,5 +523,5 @@
     <parent link="base_link"/>
     <child link="sonar_2"/>
-    <origin xyz="-0.15374 0.23214 ${0.03475+0.029}"  rpy="0 0 1.5707"/>
+    <origin xyz="0.14456 0.09192 ${0.03475+0.029}"  rpy="0 0 0"/>
   </joint>
 <!--Sonar Link2-->
@@ -530,11 +530,11 @@
       <origin xyz="0 0 0" rpy="0 0 0"/>
       <geometry>
-        <mesh filename="package://andbot_gazebo/robot_description/mesh/sonar_HC_SR04.STL"/>
-      </geometry>
-    </collision>
-    <visual>
-      <origin xyz="0 0 0" rpy="0 0 0"/>
-      <geometry>
-        <mesh filename="package://andbot_gazebo/robot_description/mesh/sonar_HC_SR04.STL"/>
+        <mesh filename="package://hyperlync_robot/robot_description/mesh/sonar_HC_SR04.STL"/>
+      </geometry>
+    </collision>
+    <visual>
+      <origin xyz="0 0 0" rpy="0 0 0"/>
+      <geometry>
+        <mesh filename="package://hyperlync_robot/robot_description/mesh/sonar_HC_SR04.STL"/>
       </geometry>
        <material name="Yellow">
@@ -559,5 +559,5 @@
     <parent link="base_link"/>
     <child link="sonar_3"/>
-    <origin xyz="-0.20374 0.20726 ${0.03475+0.029}"  rpy="0 0 1.5707"/>
+    <origin xyz="-0.10374 0.23695 ${0.03475+0.029}"  rpy="0 0 1.5707"/>
   </joint>
 <!--Sonar Link3-->
@@ -566,11 +566,11 @@
       <origin xyz="0 0 0" rpy="0 0 0"/>
       <geometry>
-        <mesh filename="package://andbot_gazebo/robot_description/mesh/sonar_HC_SR04.STL"/>
-      </geometry>
-    </collision>
-    <visual>
-      <origin xyz="0 0 0" rpy="0 0 0"/>
-      <geometry>
-        <mesh filename="package://andbot_gazebo/robot_description/mesh/sonar_HC_SR04.STL"/>
+        <mesh filename="package://hyperlync_robot/robot_description/mesh/sonar_HC_SR04.STL"/>
+      </geometry>
+    </collision>
+    <visual>
+      <origin xyz="0 0 0" rpy="0 0 0"/>
+      <geometry>
+        <mesh filename="package://hyperlync_robot/robot_description/mesh/sonar_HC_SR04.STL"/>
       </geometry>
        <material name="Yellow">
@@ -595,5 +595,5 @@
     <parent link="base_link"/>
     <child link="sonar_4"/>
-    <origin xyz="-0.25374 0.18238 ${0.03475+0.029}"  rpy="0 0 1.5707"/>
+    <origin xyz="-0.1931 0.23214 ${0.03475+0.029}"  rpy="0 0 1.5707"/>
   </joint>
 <!--Sonar Link4-->
@@ -602,11 +602,11 @@
       <origin xyz="0 0 0" rpy="0 0 0"/>
       <geometry>
-        <mesh filename="package://andbot_gazebo/robot_description/mesh/sonar_HC_SR04.STL"/>
-      </geometry>
-    </collision>
-    <visual>
-      <origin xyz="0 0 0" rpy="0 0 0"/>
-      <geometry>
-        <mesh filename="package://andbot_gazebo/robot_description/mesh/sonar_HC_SR04.STL"/>
+        <mesh filename="package://hyperlync_robot/robot_description/mesh/sonar_HC_SR04.STL"/>
+      </geometry>
+    </collision>
+    <visual>
+      <origin xyz="0 0 0" rpy="0 0 0"/>
+      <geometry>
+        <mesh filename="package://hyperlync_robot/robot_description/mesh/sonar_HC_SR04.STL"/>
       </geometry>
        <material name="Yellow">
@@ -631,5 +631,5 @@
     <parent link="base_link"/>
     <child link="sonar_5"/>
-    <origin xyz="-0.25374 -0.18238 ${0.03475+0.029}"  rpy="0 0 -1.5707"/>
+    <origin xyz="-0.27047 0.20726 ${0.03475+0.029}"  rpy="0 0 1.5707"/>
   </joint>
 <!--Sonar Link5-->
@@ -638,11 +638,11 @@
       <origin xyz="0 0 0" rpy="0 0 0"/>
       <geometry>
-        <mesh filename="package://andbot_gazebo/robot_description/mesh/sonar_HC_SR04.STL"/>
-      </geometry>
-    </collision>
-    <visual>
-      <origin xyz="0 0 0" rpy="0 0 0"/>
-      <geometry>
-        <mesh filename="package://andbot_gazebo/robot_description/mesh/sonar_HC_SR04.STL"/>
+        <mesh filename="package://hyperlync_robot/robot_description/mesh/sonar_HC_SR04.STL"/>
+      </geometry>
+    </collision>
+    <visual>
+      <origin xyz="0 0 0" rpy="0 0 0"/>
+      <geometry>
+        <mesh filename="package://hyperlync_robot/robot_description/mesh/sonar_HC_SR04.STL"/>
       </geometry>
        <material name="Yellow">
@@ -667,5 +667,5 @@
     <parent link="base_link"/>
     <child link="sonar_6"/>
-    <origin xyz="-0.20374 -0.21205 ${0.03475+0.029}"  rpy="0 0 -1.5707"/>
+    <origin xyz="-0.37437 0.05695 ${0.03475+0.029}"  rpy="0 0 3.14"/>
   </joint>
 <!--Sonar Link6-->
@@ -674,11 +674,11 @@
       <origin xyz="0 0 0" rpy="0 0 0"/>
       <geometry>
-        <mesh filename="package://andbot_gazebo/robot_description/mesh/sonar_HC_SR04.STL"/>
-      </geometry>
-    </collision>
-    <visual>
-      <origin xyz="0 0 0" rpy="0 0 0"/>
-      <geometry>
-        <mesh filename="package://andbot_gazebo/robot_description/mesh/sonar_HC_SR04.STL"/>
+        <mesh filename="package://hyperlync_robot/robot_description/mesh/sonar_HC_SR04.STL"/>
+      </geometry>
+    </collision>
+    <visual>
+      <origin xyz="0 0 0" rpy="0 0 0"/>
+      <geometry>
+        <mesh filename="package://hyperlync_robot/robot_description/mesh/sonar_HC_SR04.STL"/>
       </geometry>
        <material name="Yellow">
@@ -703,5 +703,5 @@
     <parent link="base_link"/>
     <child link="sonar_7"/>
-    <origin xyz="-0.15374 -0.23214 ${0.03475+0.029}"  rpy="0 0 -1.5707"/>
+    <origin xyz="-0.37695 0 ${0.03475+0.029}"  rpy="0 0 3.14"/>
   </joint>
 <!--Sonar Link7-->
@@ -710,11 +710,11 @@
       <origin xyz="0 0 0" rpy="0 0 0"/>
       <geometry>
-        <mesh filename="package://andbot_gazebo/robot_description/mesh/sonar_HC_SR04.STL"/>
-      </geometry>
-    </collision>
-    <visual>
-      <origin xyz="0 0 0" rpy="0 0 0"/>
-      <geometry>
-        <mesh filename="package://andbot_gazebo/robot_description/mesh/sonar_HC_SR04.STL"/>
+        <mesh filename="package://hyperlync_robot/robot_description/mesh/sonar_HC_SR04.STL"/>
+      </geometry>
+    </collision>
+    <visual>
+      <origin xyz="0 0 0" rpy="0 0 0"/>
+      <geometry>
+        <mesh filename="package://hyperlync_robot/robot_description/mesh/sonar_HC_SR04.STL"/>
       </geometry>
        <material name="Yellow">
@@ -739,5 +739,5 @@
     <parent link="base_link"/>
     <child link="sonar_8"/>
-    <origin xyz="-0.10374 -0.23695 ${0.03475+0.029}"  rpy="0 0 -1.5707"/>
+    <origin xyz="-0.37437 -0.05695 ${0.03475+0.029}"  rpy="0 0 3.14"/>
   </joint>
 <!--Sonar Link8-->
@@ -746,11 +746,11 @@
       <origin xyz="0 0 0" rpy="0 0 0"/>
       <geometry>
-        <mesh filename="package://andbot_gazebo/robot_description/mesh/sonar_HC_SR04.STL"/>
-      </geometry>
-    </collision>
-    <visual>
-      <origin xyz="0 0 0" rpy="0 0 0"/>
-      <geometry>
-        <mesh filename="package://andbot_gazebo/robot_description/mesh/sonar_HC_SR04.STL"/>
+        <mesh filename="package://hyperlync_robot/robot_description/mesh/sonar_HC_SR04.STL"/>
+      </geometry>
+    </collision>
+    <visual>
+      <origin xyz="0 0 0" rpy="0 0 0"/>
+      <geometry>
+        <mesh filename="package://hyperlync_robot/robot_description/mesh/sonar_HC_SR04.STL"/>
       </geometry>
        <material name="Yellow">
@@ -765,4 +765,148 @@
   </link>
   <gazebo reference="sonar_link8">
+    <mu1 value="2.0"/>
+    <mu2 value="2.0"/>
+    <kp value="10000000.0"/>
+    <kd value="1.0"/>
+    <material>Gazebo/Yellow</material>
+  </gazebo>
+  <!-- Base link / sonar9 link joint -->
+  <joint name="sonar_9_fixed" type="fixed">
+    <parent link="base_link"/>
+    <child link="sonar_9"/>
+    <origin xyz="-0.27047 -0.21205 ${0.03475+0.029}"  rpy="0 0 -1.5707"/>
+  </joint>
+<!--Sonar Link9-->
+  <link name="sonar_9">
+    <collision>
+      <origin xyz="0 0 0" rpy="0 0 0"/>
+      <geometry>
+        <mesh filename="package://hyperlync_robot/robot_description/mesh/sonar_HC_SR04.STL"/>
+      </geometry>
+    </collision>
+    <visual>
+      <origin xyz="0 0 0" rpy="0 0 0"/>
+      <geometry>
+        <mesh filename="package://hyperlync_robot/robot_description/mesh/sonar_HC_SR04.STL"/>
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