Commit message: daily update

File: andbot1dot2/modeldescription/urdf/andbot1dot2.xacro (robot description, xacro)
@@ -8,11 +8,11 @@
         <xacro:include filename="$(find andbot1dot2)/modeldescription/urdf/sensors/rplidar_laser.urdf.xacro" />
         <xacro:include filename="$(find andbot1dot2)/modeldescription/urdf/sensors/mpu6050_imu.urdf.xacro" />
-<link name="${robotname}_base">
+		<link name="${robotname}_base">
                 <collision>
                         <geometry>
-                                <mesh filename="package://andbot1dot2/modeldescription/mesh/andbot1dot2_housing.STL"></mesh></geometry></collision>
+                                <mesh filename="package://andbot1dot2/modeldescription/mesh/andbot1dot2_baseplate.STL"></mesh></geometry></collision>
                 <visual>
                         <geometry>
-                                <mesh filename="package://andbot1dot2/modeldescription/mesh/andbot1dot2_housing.STL"/>
+                                <mesh filename="package://andbot1dot2/modeldescription/mesh/andbot1dot2_baseplate.STL"/>
                         </geometry>
                         <material name="blue"></material>
@@ -24,21 +24,5 @@
                 </inertial>
         </link>
-<link name="${robotname}_shaft">
-                <collision>
-                        <geometry>
-                                <mesh filename="package://andbot1dot2/modeldescription/mesh/andbot1dot2_shaftholder.STL"></mesh></geometry></collision>
-                <visual>
-                        <geometry>
-                                <mesh filename="package://andbot1dot2/modeldescription/mesh/andbot1dot2_shaftholder.STL"/>
-                        </geometry>
-                        <material name="white">
-                        </material>
-                </visual>
-                <inertial>
-                        <mass value="0.2645"/>
-                        <inertia ixx="0.0014" ixy="0.0" ixz="0.0" iyy="0.0001" iyz="0.0" izz="0.0014"/>
-                </inertial>
-        </link>
-<link name="${robotname}_leftwheel">
+		<link name="${robotname}_leftwheel">
                 <collision>
                         <geometry>
@@ -52,9 +36,9 @@
                 </visual>
                 <inertial>
-                        <mass value="0.3871"/>
-                        <inertia ixx="0.0238" ixy="0.0" ixz="0.0" iyy="0.0003" iyz="0.0" izz="0.0238"/>
+                        <mass value="1.158"/><!-- Is this actually right? -->
+                        <inertia ixx="0.0532" ixy="0.0" ixz="0.0" iyy="0.0038" iyz="0.0" izz="0.0532"/>
                 </inertial>
         </link>
-<link name="${robotname}_rightwheel">
+		<link name="${robotname}_rightwheel">
                 <collision>
                         <geometry>
@@ -68,28 +52,23 @@
                 </visual>
                 <inertial>
-                        <mass value="0.3871"/>
-                        <inertia ixx="0.0238" ixy="0.0" ixz="0.0" iyy="0.0003" iyz="0.0" izz="0.0238"/>
+                        <mass value="1.158"/>
+                        <inertia ixx="0.0532" ixy="0.0" ixz="0.0" iyy="0.0038" iyz="0.0" izz="0.0532"/>
                 </inertial>
         </link>
-<joint name="base2shaft" type="fixed">
+        <joint name="base2leftwheel" type="continuous">
                 <parent link="${robotname}_base"/>
-                <child link="${robotname}_shaft"/>
-                <origin xyz="0.07 0 0.0255"/>
-        </joint>
-        <joint name="shaft2leftwheel" type="continuous">
-                <parent link="${robotname}_shaft"/>
                 <child link="${robotname}_leftwheel"/>
-                <origin xyz="0 0.1235 0"/>
+                <origin xyz="0 0.20684 0"/>
                 <axis xyz="0 -1 0"/>
         </joint>
-        <joint name="shaft2rightwheel" type="continuous">
-                <parent link="${robotname}_shaft"/>
+        <joint name="base2rightwheel" type="continuous">
+                <parent link="${robotname}_base"/>
                 <child link="${robotname}_rightwheel"/>
-                <origin xyz="0 -0.1235 0"/>
+                <origin xyz="0 -0.20684 0"/>
                 <axis xyz="0 1 0"/>
         </joint>
-        <xacro:rplidar_laser name="${robotname}" parent="${robotname}_base" ros_topic="scan" update_rate="40" min_angle="-1.3962634" max_angle="1.3962634" >
+    <xacro:rplidar_laser name="${robotname}" parent="${robotname}_base" ros_topic="scan" update_rate="40" min_angle="-1.3962634" max_angle="1.3962634" >
     </xacro:rplidar_laser>
     <xacro:mpu6050_imu name="${robotname}" parent="${robotname}_base">
     </xacro:mpu6050_imu>
-<\robot>
+</robot>

File: andbot1dot2/modeldescription/urdf/sensors/rplidar_laser.urdf.xacro (robot description, xacro)
@@ -5,18 +5,18 @@
 			<parent link="${parent}"></parent>
 			<child link="${name}_rplidar"></child>
-			<!--  rotate z axis 180 degree according to the placement on angelbot -->
-			<origin xyz="-0.0007 0.00015 0.15949" rpy="0 0 3.1415"></origin>
+			<!--  rotate z axis 180 degree according to the placement on andbot -->
+			<origin xyz="-0.02426 0.0 0.17395" rpy="0 0 0"></origin>
 		</joint>
 	  	<link name="${name}_rplidar">
 			<collision>
 				<geometry>
-					<mesh filename="package://angelbot/modeldescription/mesh/angel_rplidar.STL"></mesh></geometry></collision>
+					<mesh filename="package://andbot1dot2/modeldescription/mesh/andbot1dot2_rplidar.STL"></mesh></geometry></collision>
 			<visual>
 				<geometry>
-					<mesh filename="package://angelbot/modeldescription/mesh/angel_rplidar.STL"></mesh></geometry>
+					<mesh filename="package://andbot1dot2/modeldescription/mesh/andbot1dot2_rplidar.STL"></mesh></geometry>
 				<material name="red"></material></visual>
 			<inertial>
-				<mass value="0.20856"></mass>
-				<inertia ixx="0.0001" ixy="0.0" ixz="0.0" iyy="0.0002" iyz="0.0" izz="0.0002"></inertia></inertial>
+				<mass value="0.1646"></mass>
+				<inertia ixx="0.0046" ixy="0.0" ixz="-0.0007" iyy="0.0048" iyz="0.0" izz="0.0003"></inertia></inertial>
 		</link>
     </xacro:macro>
