Commit message: update

File: andbot/robot_description/urdf/andbot.xacro (robot description, xacro)
@@ -18,1485 +18,26 @@
   <link name="base_footprint"/>
   <link name="xv11">
-    <collision>
-      <origin xyz="0 0 -0.019" rpy="1.57 0 -1.57"/>
-      <geometry>
-        <mesh filename="package://andbot/robot_description/mesh/lidar_XV-11.STL"/>
-      </geometry>
-    </collision>
-    <visual>
-      <origin xyz="0 0 -0.019" rpy="1.57 0 -1.57"/>
-      <geometry>
-        <mesh filename="package://andbot/robot_description/mesh/lidar_XV-11.STL"/>
-      </geometry>
-       <material name="Green">
-         <color rgba="0 0 1 1"/>
-       </material>
-    </visual>
-    <inertial>
-      <origin xyz="0 0 0.07" rpy="0 0 0"/>
-      <mass value="0.1"/>
-      <inertia ixx="0.2" ixy="0" ixz="0" iyy="0.2" iyz="0" izz="0.3"/>
-    </inertial>
   </link>
-  <gazebo reference="xv11">
-    <material>Gazebo/Green</material>
-  </gazebo>
   <joint name="xv11_fixed" type="fixed">
     <parent link="base_footprint"/>
     <child link="xv11"/>
 <!--    plastic model     -->
-<origin xyz="-0.022 0 ${radius_wheel+0.135}" rpy="0 0 0"/>
+  <origin xyz="-0.022 0 ${radius_wheel+0.135}" rpy="0 0 0"/>
 <!--	metal model	-->
 <!--	<origin xyz="0.07 0 ${radius_wheel+0.135}" rpy="0 0 0"/>-->
   </joint>
-<joint name="IMU_joint" type="fixed">
+  <joint name="IMU_joint" type="fixed">
     <axis xyz="1 0 0"/>
         <origin xyz="0.0 0.0 0.055"/>
 	    <parent link="base_link"/>
 	    <child link="IMU_link"/>
-</joint>
-<link name="IMU_link">
-  <inertial>
-      <mass value="0.001"/>
-          <origin rpy="0 0 0" xyz="0 0 0"/>
-	      <inertia ixx="0.0001" ixy="0" ixz="0" iyy="0.000001" iyz="0" izz="0.0001"/>
-  </inertial>
-  <visual>
-	<origin rpy="0 0 0" xyz="0 0 0"/>
-          <geometry>
-	       <box size="0.01 0.01 0.01"/>
-	  </geometry>
-        <material name="red"/>
-	  </visual>
-	    <collision>
-	    <origin rpy="0 0 0" xyz="0 0 0"/>
-		 <geometry>
-	          <box size=".01 .01 .01"/>
-		 </geometry>
-	    </collision>
-</link>
+  </joint>
+  <link name="IMU_link"/>
 <!-- Base link -->
-  <link name="base_link">
-    <collision>
-      <origin xyz="0 0 ${radius_wheel-height_wheels_from_base}" rpy="0 0 0"/>
-      <geometry>
-        <mesh filename="package://andbot/robot_description/mesh/base_part.STL"/>
-      </geometry>
-    </collision>
-    <visual>
-      <origin xyz="0 0 ${radius_wheel-height_wheels_from_base}" rpy="0 0 0"/>
-      <geometry>
-        <mesh filename="package://andbot/robot_description/mesh/base_part.STL"/>
-      </geometry>
-       <material name="Orange">
-         <color rgba="1 0.5 0 1"/>
-       </material>
-    </visual>
-    <inertial>
-      <origin xyz="0 0 0.07" rpy="0 0 0"/>
-      <mass value="52"/>
-      <inertia ixx="0.248" ixy="0" ixz="0" iyy="0.748" iyz="0" izz="0.748"/>
-    </inertial>
-  </link>
-  <gazebo reference="base_link">
-    <material>Gazebo/Orange</material>
-  </gazebo>
-  <!-- Base footprint link / Base link joint -->
+  <link name="base_link"/>
+<!-- Base footprint link / Base link joint -->
   <joint name="base_joint" type="fixed">
     <parent link="base_footprint"/>
     <child link="base_link"/>
   </joint>
-   <!-- Caster wheel link -->
-  <link name="caster_wheel">
-    <collision>
-      <origin xyz="0 0 0" rpy="0 0 0"/>
-      <geometry>
-        <sphere radius="0.02"/>
-      </geometry>
-    </collision>
-    <visual>
-      <origin xyz="0 0 0" rpy="0 0 0"/>
-      <geometry>
-        <sphere radius="0.02"/>
-      </geometry>
-       <material name="White">
-         <color rgba="1 0 0 1"/>
-       </material>
-    </visual>
-    <inertial>
-      <origin xyz="0 0 0" rpy="0 0 0"/>
-      <mass value="0.05"/>
-      <inertia ixx="0.0098" ixy="0" ixz="0" iyy="0.0098" iyz="0" izz="0.0098"/>
-    </inertial>
-  </link>
-  <gazebo reference="caster_wheel">
-    <mu1>0.04</mu1>
-    <mu2>0.04</mu2>
-    <material>Gazebo/White</material>
-  </gazebo>
-  <!-- Base link / Caster wheel joint -->
-  <joint name="fixed" type="fixed">
-    <parent link="base_link"/>
-    <child link="caster_wheel"/>
-    <origin xyz="-0.3 0 0.02" rpy="0 0 0"/>
-  </joint>
-  <!-- Body link -->
-<!--
-  <link name="body_link">
-    <collision>
-      <origin xyz="0 0 0" rpy="0 0 0"/>
-      <geometry>
-        <mesh filename="package://andbot/robot_description/mesh/fake_body.STL"/>
-      </geometry>
-    </collision>
-    <visual>
-      <origin xyz="0 0 0" rpy="0 0 0"/>
-      <geometry>
-        <mesh filename="package://andbot/robot_description/mesh/fake_body.STL"/>
-      </geometry>
-       <material name="Blue">
-       </material>
-    </visual>
-    <inertial>
-      <origin xyz="0 0 0.00" rpy="0 0 0"/>
-      <mass value="3.5"/>
-      <inertia ixx="0.248" ixy="0" ixz="0" iyy="0.248" iyz="0" izz="0.748"/>
-    </inertial>
-  </link>
-  <gazebo reference="body_link">
-    <material>Gazebo/Blue</material>
-  </gazebo>
-  <joint name="body_joint" type="fixed">
-    <parent link="base_link"/>
-    <child link="body_link"/>
-    <origin xyz="0 0 0.029" rpy="0 0 0"/>
-  </joint>
--->
-  <!-- Head link -->
-  <link name="head_link">
-    <collision>
-      <origin xyz="0 0 0" rpy="0 0 0"/>
-      <geometry>
-        <mesh filename="package://andbot/robot_description/mesh/head.STL"/>
-      </geometry>
-    </collision>
-    <visual>
-      <origin xyz="0 0 0" rpy="0 0 0"/>
-      <geometry>
-        <mesh filename="package://andbot/robot_description/mesh/head.STL"/>
-      </geometry>
-       <material name="Blue">
-         <color rgba="0 0 1 0.5"/>
-       </material>
-    </visual>
-    <inertial>
-      <origin xyz="0 0 0.0" rpy="0 0 0"/>
-      <mass value="1.5"/>
-      <inertia ixx="0.248" ixy="0" ixz="0" iyy="0.248" iyz="0" izz="0.008"/>
-    </inertial>
-  </link>
-  <gazebo reference="head_link">
-    <material>Gazebo/Blue</material>
-  </gazebo>
-  <!-- Base link /Head Link joint -->
-  <joint name="head_joint" type="continuous">
-    <parent link="base_link"/>
-    <child link="head_link"/>
-    <origin xyz="-0.145 0 1.075" rpy="0 0 0"/>
-    <axis xyz="0 0 1"/>
-          <limit upper="1.57" lower="-1.57" velocity="10" effort="7"/>
-	  <joint_properties damping="0.0" friction="0.0"/>
-  </joint>
-  <!-- Transmission for laser joint -->
-  <transmission name="head_trans">
-    <type>transmission_interface/SimpleTransmission</type>
-    <joint name="head_joint">
-      <hardwareInterface>EffortJointInterface</hardwareInterface>
-    </joint>
-    <actuator name="headMotor">
-      <hardwareInterface>EffortJointInterface</hardwareInterface>
-      <mechanicalWhiteuction>1</mechanicalWhiteuction>
-    </actuator>
-  </transmission>
-  <!-- left_arm_link1 link -->
-  <link name="left_arm_link1">
-    <collision>
-      <origin xyz="0 0 0" rpy="-1.5707 1.5707 0"/>
-      <geometry>
-        <mesh filename="package://andbot/robot_description/mesh/arm_link1.STL"/>
-      </geometry>
-    </collision>
-    <visual>
-      <origin xyz="0 0 0" rpy="-1.5707 1.5707 0"/>
-      <geometry>
-        <mesh filename="package://andbot/robot_description/mesh/arm_link1.STL"/>
-      </geometry>
-       <material name="Blue">
-         <color rgba="0 0 1 0.5"/>
-       </material>
-    </visual>
-    <inertial>
-      <origin xyz="0 0 0.00" rpy="0 0 0"/>
-      <mass value="0.75"/>
-      <inertia ixx="0.148" ixy="0" ixz="0" iyy="0.148" iyz="0" izz="0.748"/>
-    </inertial>
-  </link>
-  <gazebo reference="left_arm_link1">
-    <material>Gazebo/Blue</material>
-  </gazebo>
-  <!-- Base link /left_arm_link1 Link joint -->
-  <joint name="left_arm_link1_joint" type="fixed">
-    <parent link="base_link"/>
-    <child link="left_arm_link1"/>
-    <origin xyz="-0.145 0.185 0.909" rpy="0 0 0"/>
-  </joint>
-  <!-- Left left_arm_link2 link -->
-  <link name="left_arm_link2">
-    <collision>
-      <origin xyz="0 0 0" rpy="-1.5707 1.5707 0"/>
-      <geometry>
-        <mesh filename="package://andbot/robot_description/mesh/arm_link2.STL"/>
-      </geometry>
-    </collision>
-    <visual>
-      <origin xyz="0 0 0" rpy="-1.5707 1.5707 0"/>
-      <geometry>
-        <mesh filename="package://andbot/robot_description/mesh/arm_link2.STL"/>
-      </geometry>
-       <material name="Blue">
-         <color rgba="0 0 1 0.5"/>
-       </material>
-    </visual>
-    <inertial>
-      <origin xyz="0 0 0.00" rpy="0 0 0"/>
-      <mass value="0.75"/>
-      <inertia ixx="0.148" ixy="0" ixz="0" iyy="0.148" iyz="0" izz="0.748"/>
-    </inertial>
-  </link>
-  <gazebo reference="left_arm_link2">
-    <material>Gazebo/Blue</material>
-  </gazebo>
-  <!-- Base link /Left_arm_link2 Link joint -->
-  <joint name="left_arm_link2_joint" type="fixed">
-    <parent link="left_arm_link1"/>
-    <child link="left_arm_link2"/>
-    <origin xyz="0 0 -0.205" rpy="0 0 0"/>
-  </joint>
-  <!-- right_arm_link1 link -->
-  <link name="right_arm_link1">
-    <collision>
-      <origin xyz="0 0 0" rpy="1.57 1.5707 0"/>
-      <geometry>
-        <mesh filename="package://andbot/robot_description/mesh/arm_link1.STL"/>
-      </geometry>
-    </collision>
-    <visual>
-      <origin xyz="0 0 0" rpy="1.57 1.5707 0"/>
-      <geometry>
-        <mesh filename="package://andbot/robot_description/mesh/arm_link1.STL"/>
-      </geometry>
-       <material name="Blue">
-         <color rgba="0 0 1 0.5"/>
-       </material>
-    </visual>
-    <inertial>
-      <origin xyz="0 0 0.00" rpy="0 0 0"/>
-      <mass value="0.75"/>
-      <inertia ixx="0.148" ixy="0" ixz="0" iyy="0.148" iyz="0" izz="0.748"/>
-    </inertial>
-  </link>
-  <gazebo reference="right_arm_link1">
-    <material>Gazebo/Blue</material>
-  </gazebo>
-  <!-- Base link /Right arm_link1 Link joint -->
-  <joint name="right_arm_link1_joint" type="fixed">
-    <parent link="base_link"/>
-    <child link="right_arm_link1"/>
-    <origin xyz="-0.145 -0.185 0.909" rpy="0 0 0"/>
-  </joint>
-  <!-- right_arm_link2 link -->
-  <link name="right_arm_link2">
-    <collision>
-      <origin xyz="0 0 0" rpy="-1.5707 1.5707 3.14"/>
-      <geometry>
-        <mesh filename="package://andbot/robot_description/mesh/arm_link2.STL"/>
-      </geometry>
-    </collision>
-    <visual>
-      <origin xyz="0 0 0" rpy="-1.5707 1.5707 0"/>
-      <geometry>
-        <mesh filename="package://andbot/robot_description/mesh/arm_link2.STL"/>
-      </geometry>
-       <material name="Blue">
-         <color rgba="0 0 1 0.5"/>
-       </material>
-    </visual>
-    <inertial>
-      <origin xyz="0 0 0.00" rpy="0 0 0"/>
-      <mass value="0.75"/>
-      <inertia ixx="0.148" ixy="0" ixz="0" iyy="0.148" iyz="0" izz="0.748"/>
-    </inertial>
-  </link>
-  <gazebo reference="right_arm_link2">
-    <material>Gazebo/Blue</material>
-  </gazebo>
-  <!-- Base link /right_arm_link2 Link joint -->
-  <joint name="right_arm_link2_joint" type="fixed">
-    <parent link="right_arm_link1"/>
-    <child link="right_arm_link2"/>
-    <origin xyz="0 0 -0.205" rpy="0 0 0"/>
-  </joint>
-  <!-- Base link / Laser link joint -->
-  <joint name="laser_joint" type="fixed">
-    <parent link="head_link"/>
-    <child link="laser"/>
-    <origin xyz="0.1 0 -0.05" rpy="0 0 0"/>
-  </joint>
-  <!-- Laser link -->
-  <link name="laser">
-    <collision>
-      <origin xyz="0 0 0" rpy="0 1.57 0"/>
-      <geometry>
-        <cylinder length="0.08" radius="0.01"/>
-      </geometry>
-    </collision>
-    <visual>
-      <origin xyz="0 0 0" rpy="0 1.57 0"/>
-      <geometry>
-        <cylinder length="0.08" radius="0.01"/>
-      </geometry>
-    </visual>
-    <inertial>
-      <mass value="0.002"/>
-      <origin xyz="0 0 0" rpy="0 0 0"/>
-      <inertia ixx="1e-6" ixy="0" ixz="0" iyy="1e-6" iyz="0" izz="0.01"/>
-    </inertial>
-  </link>
-  <gazebo reference="laser">
-    <mu1 value="5.0"/>
-    <mu2 value="5.0"/>
-    <kp value="10000000.0"/>
-    <kd value="1.0"/>
-  </gazebo>
-  <!-- Left wheel link -->
-  <link name="left_wheel">
-    <collision>
-      <origin xyz="0 0 0" rpy="0 1.570795 1.570795"/>
-      <geometry>
-        <mesh filename="package://andbot/robot_description/mesh/wheel-D152_SMALL.STL"/>
-      </geometry>
-    </collision>
-    <visual>
-      <origin xyz="0 0 0" rpy="0 1.570795 1.570795"/>
-      <geometry>
-        <mesh filename="package://andbot/robot_description/mesh/wheel-D152_SMALL.STL"/>
-      </geometry>
-       <material name="Black">
-         <color rgba="0 0 0 1"/>
-       </material>
-    </visual>
-    <inertial>
-      <origin xyz="0 0 0" rpy="0 1.570795 1.570795"/>
-      <mass value="0.4"/>
-      <inertia ixx="0.0135" ixy="0" ixz="0" iyy="0.0135" iyz="0" izz="0.025"/>
-    </inertial>
-  </link>
-  <gazebo reference="left_wheel">
-    <mu1 value="2.0"/>
-    <mu2 value="2.0"/>
-    <kp value="10000000.0"/>
-    <kd value="1.0"/>
-    <material>Gazebo/Black</material>
-  </gazebo>
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