Commit message: change 1M baud, sonar urdf

File: andbot/robot_description/urdf/andbot_sonar.xacro (robot description, xacro)
@@ -675,5 +675,7 @@
     <parent link="base_link"/>
     <child link="sonar_1"/>
-    <origin xyz="-0.37437 0.05695 ${0.03475+0.029}"  rpy="0 0 3.14"/>
+    <!--<origin xyz="-0.37437 0.05695 ${0.03475+0.029}"  rpy="0 0 3.14"/>
+    -->
+    <origin xyz="-0.37437 0.05695 ${0.03475+0.029}"  rpy="0 0 2.878200612"/>
   </joint>
 <!--Sonar Link6-->
@@ -747,5 +749,7 @@
     <parent link="base_link"/>
     <child link="sonar_3"/>
-    <origin xyz="-0.37437 -0.05695 ${0.03475+0.029}"  rpy="0 0 3.14"/>
+    <!--<origin xyz="-0.37437 -0.05695 ${0.03475+0.029}"  rpy="0 0 3.14"/>
+    -->
+    <origin xyz="-0.37437 -0.05695 ${0.03475+0.029}"  rpy="0 0 -2.878200612"/>
   </joint>
 <!--Sonar Link8-->

Commit message: replace lidar to rplidar

File: andbot/robot_description/urdf/andbot_sonar.xacro (robot description, xacro)
@@ -17,5 +17,5 @@
   <!-- Base footprint link-->
   <link name="base_footprint"/>
-  <link name="xv11">
+  <link name="rplidar">
     <collision>
       <origin xyz="0 0 -0.019" rpy="1.57 0 -1.57"/>
@@ -39,12 +39,12 @@
     </inertial>
   </link>
-  <gazebo reference="xv11">
+  <gazebo reference="rplidar">
     <material>Gazebo/Green</material>
   </gazebo>
-  <joint name="xv11_fixed" type="fixed">
+  <joint name="rplidar_fixed" type="fixed">
     <parent link="base_footprint"/>
-    <child link="xv11"/>
+    <child link="rplidar"/>
 <!--    plastic model     -->
-<origin xyz="-0.022 0 ${radius_wheel+0.135}" rpy="0 0 0"/>
+<origin xyz="-0.022 0 ${radius_wheel+0.135}" rpy="0 0 3.14"/>
 <!--	metal model	-->
 <!--	<origin xyz="0.07 0 ${radius_wheel+0.135}" rpy="0 0 0"/>-->
@@ -999,10 +999,10 @@
     </sensor>
   </gazebo>
-<!-- xv11 plugin -->
-  <gazebo reference="xv11">
+<!-- rplidar plugin -->
+  <gazebo reference="rplidar">
     <mu1>1.0</mu1>
     <mu2>1.0</mu2>
     <material>Gazebo/Blue</material>
-    <sensor type="ray" name="xv11_sensor">
+    <sensor type="ray" name="rplidar_sensor">
       <pose>0 0 0 0 0 0</pose>
       <visualize>true</visualize>
@@ -1035,6 +1035,6 @@
       </ray>
       <plugin name="gazebo_ros_head_hokuyo_controller" filename="libgazebo_ros_laser.so">
-        <topicName>xv11_scan</topicName>
-        <frameName>xv11</frameName>
+        <topicName>rplidar_scan</topicName>
+        <frameName>rplidar</frameName>
       </plugin>
     </sensor>
