Commit message: daily update.Gmapping function with or without ekf package are now workable.

File: andbot1dot2/modeldescription/urdf/sensors/mpu6050_imu.urdf.xacro (robot description, xacro)
@@ -5,5 +5,5 @@
 			<parent link="${parent}"></parent>
 			<child link="${name}_mpu6050_link"></child>
-			<origin xyz="0.07 0 0.0255" rpy="0 0 0"></origin>
+			<origin xyz="0.0 0.0 0.0" rpy="0 0 0"></origin>
 		</joint>
 	  	<link name="${name}_mpu6050_link">

File: andbot1dot2/modeldescription/urdf/sensors/rplidar_laser.urdf.xacro (robot description, xacro)
@@ -6,5 +6,5 @@
 			<child link="${name}_rplidar"></child>
 			<!--  rotate z axis 180 degree according to the placement on andbot -->
-			<origin xyz="-0.02426 0.0 0.17395" rpy="0 0 0"></origin>
+			<origin xyz="-0.02426 0.0 0.17395" rpy="0 0 3.14159"></origin>
 		</joint>
 	  	<link name="${name}_rplidar">
