Commit message: daily upload

File: angelbot/modeldescription/urdf/angelbot.xacro (robot description, xacro)
@@ -31,5 +31,5 @@
 		<inertial>
 			<mass value="0.42642"/>
-			<inertia ixx="0.0119" ixy="0.0" ixz="-0.0001" iyy="0.0035" iyz="0.0" izz="0.0063"/>
+			<inertia ixx="0.0119" ixy="0.0" ixz="0.0" iyy="0.0118" iyz="0.0" izz="0.0063"/>
 		</inertial>
 	</link>
@@ -63,5 +63,5 @@
 		<inertial>
 			<mass value="0.3871"/>
-			<inertia ixx="0.0002" ixy="0.0" ixz="0.0" iyy="0.0003" iyz="0.0" izz="0.0002"/>
+			<inertia ixx="0.0238" ixy="0.0" ixz="0.0" iyy="0.0003" iyz="0.0" izz="0.0238"/>
 		</inertial>
 	</link>
@@ -79,5 +79,5 @@
 		<inertial>
 			<mass value="0.3871"/>
-			<inertia ixx="0.0002" ixy="0.0" ixz="0.0" iyy="0.0003" iyz="0.0" izz="0.0002"/>
+			<inertia ixx="0.0238" ixy="0.0" ixz="0.0" iyy="0.0003" iyz="0.0" izz="0.0238"/>
 		</inertial>
 	</link>
@@ -96,5 +96,5 @@
 		<parent link="${robotname}_base"/>
 		<child link="${robotname}_shaft"/>
-		<origin xyz="-0.07 0 0.0255"/>
+		<origin xyz="0.07 0 0.0255"/>
 	</joint>
 	<joint name="shaft2leftwheel" type="continuous">
@@ -102,5 +102,5 @@
 		<child link="${robotname}_leftwheel"/>
 		<origin xyz="0 0.1235 0"/>
-		<axis xyz="0 1 0"/>
+		<axis xyz="0 -1 0"/>
 	</joint>
 	<joint name="shaft2rightwheel" type="continuous">
@@ -108,5 +108,5 @@
 		<child link="${robotname}_rightwheel"/>
 		<origin xyz="0 -0.1235 0"/>
-		<axis xyz="0 -1 0"/>
+		<axis xyz="0 1 0"/>
 	</joint>
 	<joint name="base2rplidar" type="fixed">

Commit message: modify urdf for laser sensor

File: angelbot/modeldescription/urdf/angelbot.xacro (robot description, xacro)
@@ -6,4 +6,5 @@
  	<!-- Import Rviz colors -->
 	<xacro:include filename="$(find angelbot)/modeldescription/urdf/angelbotmaterial4rviz.xacro"/>
+	<xacro:include filename="$(find angelbot)/modeldescription/urdf/sensors/rplidar_laser.urdf.xacro" />
 	<transmission name="trans_mobile_left">
 		<type>transmission_interface/SimpleTransmission</type>
@@ -82,15 +83,4 @@
 		</inertial>
 	</link>
-	<link name="${robotname}_rplidar">
-		<collision>
-			<geometry>
-				<mesh filename="package://angelbot/modeldescription/mesh/angel_rplidar.STL"></mesh></geometry></collision>
-		<visual>
-			<geometry>
-				<mesh filename="package://angelbot/modeldescription/mesh/angel_rplidar.STL"></mesh></geometry>
-			<material name="red"></material></visual>
-		<inertial>
-			<mass value="0.20856"></mass>
-			<inertia ixx="0.0001" ixy="0.0" ixz="0.0" iyy="0.0002" iyz="0.0" izz="0.0002"></inertia></inertial></link>
 	<joint name="base2shaft" type="fixed">
 		<parent link="${robotname}_base"/>
@@ -110,7 +100,5 @@
 		<axis xyz="0 1 0"/>
 	</joint>
-	<joint name="base2rplidar" type="fixed">
-		<parent link="${robotname}_base"></parent>
-		<child link="${robotname}_rplidar"></child>
-		<origin xyz="-0.0007 0.00015 0.15949"></origin></joint>
+	<xacro:rplidar_laser name="${robotname}" parent="${robotname}_base" ros_topic="/scan" update_rate="40" min_angle="-1.3962634" max_angle="1.3962634" >
+    </xacro:rplidar_laser>
 </robot>

Commit message: modify urdf. wrong assigning origin of differential drive

File: angelbot/modeldescription/urdf/angelbot.xacro (robot description, xacro)
@@ -20,5 +20,5 @@
 		<actuator name="rightwheelmotor">
 			<mechanicalReduction>1</mechanicalReduction></actuator></transmission>
-	<link name="${robotname}_base">
+	<link name="${robotname}_housing">
 		<collision>
 			<geometry>
@@ -36,5 +36,5 @@
 		</inertial>
 	</link>
-	<link name="${robotname}_shaft">
+	<link name="${robotname}_base">
 		<collision>
 			<geometry>
@@ -84,17 +84,17 @@
 		</inertial>
 	</link>
-	<joint name="base2shaft" type="fixed">
+	<joint name="base2housing" type="fixed">
 		<parent link="${robotname}_base"/>
-		<child link="${robotname}_shaft"/>
-		<origin xyz="0.07 0 0.0255"/>
+		<child link="${robotname}_housing"/>
+		<origin xyz="-0.07 0 -0.0255"/>
 	</joint>
-	<joint name="shaft2leftwheel" type="continuous">
-		<parent link="${robotname}_shaft"/>
+	<joint name="base2leftwheel" type="continuous">
+		<parent link="${robotname}_base"/>
 		<child link="${robotname}_leftwheel"/>
 		<origin xyz="0 0.1235 0"/>
 		<axis xyz="0 -1 0"/>
 	</joint>
-	<joint name="shaft2rightwheel" type="continuous">
-		<parent link="${robotname}_shaft"/>
+	<joint name="base2rightwheel" type="continuous">
+		<parent link="${robotname}_base"/>
 		<child link="${robotname}_rightwheel"/>
 		<origin xyz="0 -0.1235 0"/>

File: angelbot/modeldescription/urdf/sensors/mpu6050_imu.urdf.xacro (robot description, xacro)
@@ -5,5 +5,5 @@
 			<parent link="${parent}"></parent>
 			<child link="${name}_mpu6050_link"></child>
-			<origin xyz="0.07 0 0.0255" rpy="0 0 0"></origin>
+			<origin xyz="0 0 -0.0155" rpy="0 0 0"></origin>
 		</joint>
 	  	<link name="${name}_mpu6050_link">

File: angelbot/modeldescription/urdf/sensors/rplidar_laser.urdf.xacro (robot description, xacro)
@@ -6,5 +6,5 @@
 			<child link="${name}_rplidar"></child>
 			<!--  rotate z axis 180 degree according to the placement on angelbot -->
-			<origin xyz="-0.0007 0.00015 0.15949" rpy="0 0 3.1415"></origin>
+			<origin xyz="-0.0707 0.00015 0.13399" rpy="0 0 3.1415"></origin>
 		</joint>
 	  	<link name="${name}_rplidar">

Commit message: correct urdf

File: angelbot/modeldescription/urdf/angelbot.xacro (robot description, xacro)
@@ -92,5 +92,5 @@
 		<parent link="${robotname}_base"/>
 		<child link="${robotname}_leftwheel"/>
-		<origin xyz="0 0.1235 0"/>
+		<origin xyz="0 0.1227 0"/>
 		<axis xyz="0 -1 0"/>
 	</joint>
@@ -98,5 +98,5 @@
 		<parent link="${robotname}_base"/>
 		<child link="${robotname}_rightwheel"/>
-		<origin xyz="0 -0.1235 0"/>
+		<origin xyz="0 -0.1227 0"/>
 		<axis xyz="0 1 0"/>
 	</joint>

File: angelbot/modeldescription/urdf/sensors/rplidar_laser.urdf.xacro (robot description, xacro)
@@ -6,5 +6,5 @@
 			<child link="${name}_rplidar"></child>
 			<!--  rotate z axis 180 degree according to the placement on angelbot -->
-			<origin xyz="-0.0707 0.00015 0.13399" rpy="0 0 3.1415"></origin>
+			<origin xyz="0.0376 0.00015 0.128" rpy="0 0 3.1415"></origin>
 		</joint>
 	  	<link name="${name}_rplidar">

Commit message: store files

File: angelbot/modeldescription/urdf/angelbot.xacro (robot description, xacro)
@@ -39,8 +39,8 @@
 		<collision>
 			<geometry>
-				<mesh filename="package://angelbot/modeldescription/mesh/angel_shaftholder.STL"></mesh></geometry></collision>
+				<mesh filename="package://angelbot/modeldescription/mesh/rugby_base.STL"></mesh></geometry></collision>
 		<visual>
 			<geometry>
-				<mesh filename="package://angelbot/modeldescription/mesh/angel_shaftholder.STL"/>
+				<mesh filename="package://angelbot/modeldescription/mesh/rugby_base.STL"/>
 			</geometry>
 			<material name="white">
