Commit message: xacro name change

File: rugby/modeldescription/urdf/rugby.xacro (robot description, xacro)
@@ -1,9 +1,9 @@
 <?xml version="1.0"?>
-<robot xmlns:xacro="http://www.ros.org/wiki/xacro" name="angelbot">
-	<xacro:property name="robotname" value="angelbot"/>
+<robot xmlns:xacro="http://www.ros.org/wiki/xacro" name="rugby">
+	<xacro:property name="robotname" value="rugby"/>
 	<!-- Import all Gazebo-customization elements, including Gazebo colors-->
- 	<xacro:include filename="$(find rugby)/modeldescription/urdf/angelbot.gazebo" />
+ 	<xacro:include filename="$(find rugby)/modeldescription/urdf/rugby.gazebo" />
  	<!-- Import Rviz colors -->
-	<xacro:include filename="$(find rugby)/modeldescription/urdf/angelbotmaterial4rviz.xacro"/>
+	<xacro:include filename="$(find rugby)/modeldescription/urdf/rugbymaterial4rviz.xacro"/>
 	<xacro:include filename="$(find rugby)/modeldescription/urdf/sensors/rplidar_laser.urdf.xacro" />
 	<xacro:include filename="$(find rugby)/modeldescription/urdf/sensors/mpu6050_imu.urdf.xacro" />
@@ -23,8 +23,8 @@
 		<collision>
 			<geometry>
-				<mesh filename="package://angelbot/modeldescription/mesh/angel_housing.STL"></mesh></geometry></collision>
+				<mesh filename="package://rugby/modeldescription/mesh/angel_housing.STL"></mesh></geometry></collision>
 		<visual>
 			<geometry>
-				<mesh filename="package://angelbot/modeldescription/mesh/angel_housing.STL"/>
+				<mesh filename="package://rugby/modeldescription/mesh/angel_housing.STL"/>
 			</geometry>
 			<material name="blue"></material>
@@ -39,8 +39,8 @@
 		<collision>
 			<geometry>
-				<mesh filename="package://angelbot/modeldescription/mesh/rugby_base.STL"></mesh></geometry></collision>
+				<mesh filename="package://rugby/modeldescription/mesh/rugby_base.STL"></mesh></geometry></collision>
 		<visual>
 			<geometry>
-				<mesh filename="package://angelbot/modeldescription/mesh/rugby_base.STL"/>
+				<mesh filename="package://rugby/modeldescription/mesh/rugby_base.STL"/>
 			</geometry>
 			<material name="white">
@@ -55,8 +55,8 @@
 		<collision>
 			<geometry>
-				<mesh filename="package://angelbot/modeldescription/mesh/angel_leftwheel.STL"></mesh></geometry></collision>
+				<mesh filename="package://rugby/modeldescription/mesh/angel_leftwheel.STL"></mesh></geometry></collision>
 		<visual>
 			<geometry>
-				<mesh filename="package://angelbot/modeldescription/mesh/angel_leftwheel.STL"/>
+				<mesh filename="package://rugby/modeldescription/mesh/angel_leftwheel.STL"/>
 			</geometry>
 			<material name="grey">
@@ -71,8 +71,8 @@
 		<collision>
 			<geometry>
-				<mesh filename="package://angelbot/modeldescription/mesh/angel_rightwheel.STL"></mesh></geometry></collision>
+				<mesh filename="package://rugby/modeldescription/mesh/angel_rightwheel.STL"></mesh></geometry></collision>
 		<visual>
 			<geometry>
-				<mesh filename="package://angelbot/modeldescription/mesh/angel_rightwheel.STL"/>
+				<mesh filename="package://rugby/modeldescription/mesh/angel_rightwheel.STL"/>
 			</geometry>
 			<material name="grey">
