Commit message: test

File: rugby/modeldescription/urdf/sensors/mpu6050_imu.urdf.xacro (robot description, xacro)
@@ -3,9 +3,9 @@
   	<xacro:macro name="mpu6050_imu" params="name parent">
 	  	<joint name="base2mpu6050" type="fixed">
-			<parent link="${parent}"></parent>
-			<child link="${name}_mpu6050_link"></child>
+			<parent link="rugby_base"></parent>
+			<child link="rugby_mpu6050_link"></child>
 			<origin xyz="0 0 -0.0155" rpy="0 0 0"></origin>
 		</joint>
-	  	<link name="${name}_mpu6050_link">
+	  	<link name="rugby_mpu6050_link">
 			<collision>
 				<geometry>

File: rugby/modeldescription/urdf/sensors/rplidar_laser.urdf.xacro (robot description, xacro)
@@ -3,10 +3,10 @@
   	<xacro:macro name="rplidar_laser" params="name parent ros_topic update_rate min_angle max_angle">
 	  	<joint name="base2rplidar" type="fixed">
-			<parent link="${parent}"></parent>
-			<child link="${name}_rplidar"></child>
+			<parent link="rugby_base"></parent>
+			<child link="rugby_rplidar"></child>
 			<!--  rotate z axis 180 degree according to the placement on angelbot -->
 			<origin xyz="0.0376 0.00015 0.128" rpy="0 0 3.1415"></origin>
 		</joint>
-	  	<link name="${name}_rplidar">
+	  	<link name="rugby_rplidar">
 			<collision>
 				<geometry>
